Commit message: 1014 遇到了额外的碰撞问题，准备换xml文件导入

File: assets/l3/l3_29dof_neck_fixed.urdf (robot description, URDF)
Before this commit: robot l3-4_29dof_0612_neck_fixed, 51 links, 50 joints
Links:
- added link chest_in_torso
Joints:
- added joint chest_in_torso_joint: type fixed, parent torso_base_link, child chest_in_torso, origin xyz=-0.03959 -0.00224 0.14792 rpy=0 0 0

Commit message: 1017对照了urdf，还是有碰撞问题

File: assets/l3/l3_29dof_neck_fixed.urdf (robot description, URDF)
Before this commit: robot l3-4_29dof_0612_neck_fixed, 52 links, 51 joints
Links:
- removed link chest_in_torso
Joints:
- removed joint chest_in_torso_joint
